Commit message: switched base of hand one joint further up

File: hose_localization/gripper_descriptions/left_gripper_v3.urdf (robot description, URDF)
Before this commit: robot drchubo_left_gripper_v3, 11 links, 10 joints
Links:
- added link Body_LWP, mass 0.327632198289; collision mesh filename=package://drchubo_v3/meshes/convhull_LWP_merged.stl; visual mesh filename=package://drchubo_v3/meshes/convhull_LWP_merged.stl
Joints:
- added joint LWR: type revolute, parent Body_LWP, child Body_LWR, origin xyz=0.027 -0.067 0 rpy=0 0 0, axis -1.0 0 0, limit lower=-2.69956074975 upper=2.7000516236 effort=25 velocity=6.28318530718

File: hose_localization/gripper_descriptions/right_gripper_v3.urdf (robot description, URDF)
Before this commit: robot drchubo_right_gripper_v3, 14 links, 13 joints
Links:
- added link Body_RWP, mass 0.327632198289; collision mesh filename=package://drchubo_v3/meshes/convhull_RWP_merged.stl; visual mesh filename=package://drchubo_v3/meshes/convhull_RWP_merged.stl
Joints:
- added joint RWR: type revolute, parent Body_RWP, child Body_RWR, origin xyz=0.027 0.067 0 rpy=0 0 0, axis -1.0 0 0, limit lower=-2.69195220504 upper=2.70766016831 effort=25 velocity=6.28318530718
